File: Programmable DC Load.brd (EAGLE design)
At the start: 94 x 94.9 mm, 42 parts, among them IC1 LM2596S, IC3 LM358N, J2 POWER_JACK, Q1 IRF540, U1 ATMEGA328PB-AU, X1 332-02

Commit message: Add files via upload
Parts:
- removed IC3: LM358N, linear:DIL08
- removed J2: POWER_JACK, SparkFun-Connectors:POWER_JACK_PTH
- removed R15: POTENTIOMETER, pot:3223G
- added IC2: LM358MX, linear:SO08
- added POT1: RK09K1130A5R, RK09K1130A5R:RK09K1130A5R
- added U$6: 2.1MMJACKTHM, ECE388:PJ-102A
- DECREASE, INCREASE: value MOMENTARYBUTTON -> EVP-BFAC1A000; device ECE388:SPST_NO_SMD -> EVP-BFAC1A000:EVPBFAC1A000
- U$1: value MCP4921-E/P -> MCP4921-E/SN; device MCP4921-E_P:DIP787W46P254L927H533Q8 -> MCP4921-E_SN:SOIC127P600X175-8N
- moved U$2 90.3 mm to (95.2, 92.7)
- moved R9 18.8 mm to (43.2, 14.0), turned to 90 degrees
- moved R11 16.6 mm to (61.0, 14.0), turned to 90 degrees
- moved DECREASE 13.3 mm to (34.3, 12.7)
- moved INCREASE 10.9 mm to (52.1, 12.7)
- moved C6 8.52 mm to (52.1, 3.81), turned to 0 degrees
- moved C7 7.73 mm to (34.3, 3.81), turned to 0 degrees
- moved U$1 6.84 mm to (68.6, 21.6)
- moved Q1 6.48 mm to (87.6, 47.0)
- moved C1 5.39 mm to (74.9, 17.8)
- moved R4 5.08 mm to (66.0, 38.1)
- moved R1 4.58 mm to (41.9, 25.4)
- moved R10 3.81 mm to (92.7, 81.3)
- moved T1 3.59 mm to (90.2, 12.7)
- moved X1 3.59 mm to (94.0, 6.35)
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Connections:
- net +12V: now also IC2.8, U$6.TIP; no longer IC3.8, J2.PWR
- net +5V: now also POT1.VCC; no longer R15.1
- net CURRENT_SENSE: now also IC2.7; no longer IC3.7
- net GND: now also DECREASE.A1, IC2.4, INCREASE.A1, POT1.GND, U$6.RING, U$6.RING_SW; no longer DECREASE.1, IC3.4, INCREASE.1, J2.GND, J2.GNDBREAK, R15.3
- net N$10: now also IC2.3; no longer IC3.3
- net N$12: now also POT1.OUT; no longer R15.2
- net N$16: now also IC2.1; no longer IC3.1
- net N$19: now also IC2.2, IC2.5; no longer IC3.2, IC3.5
- net N$22: now also IC2.6; no longer IC3.6
- net N$6: now also DECREASE.B1; no longer DECREASE.3
- net N$8: now also INCREASE.B1; no longer INCREASE.3
Routing:
- net SCK: track 12.4 -> 29.7 mm
- net N$18: track 27.6 -> 13.5 mm
- net N$20: track 60.0 -> 47.9 mm
- net N$21: track 57.9 -> 67.9 mm
- net N$23: track 5.16 -> 14.5 mm
- net RESET: track 57.7 -> 49.5 mm
- net +12V: track 127.5 -> 120.7 mm
- net CS: track 15.7 -> 22.0 mm
- net +5V: track 274.0 -> 268.1 mm, vias 4 -> 5
- net N$24: track 5.09 -> 10.9 mm
- net N$10: track 10.6 -> 16.1 mm
- net N$16: track 14.6 -> 19.1 mm
- net SDI: track 16.4 -> 20.6 mm
- net CURRENT_SENSE: track 46.0 -> 50.2 mm
- net N$19: track 30.0 -> 27.3 mm
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Other:
- board size 94 x 94.9 mm -> 97.8 x 94.9 mm
- board text added: "DC Programmable Load V3"
- board text removed: "DC Programmable Load V2"

Commit message: Add files via upload
Parts:
- moved C7 1.27 mm to (35.6, 3.81)
Routing:
- net PC5: track 52.1 -> 50.9 mm
