File: Programmable DC Load.sch (EAGLE design)
At the start: 42 parts, among them IC1 LM2596S, IC3 LM358N, J2 POWER_JACK, Q1 IRF540, U1 ATMEGA328PB-AU, X1 332-02

Commit message: Add files via upload
Parts:
- removed IC3: LM358N, linear:LM358N
- removed J2: POWER_JACK, SparkFun-Connectors:POWER_JACK
- removed R15: POTENTIOMETER, pot:TRIM_EU-3223G
- added IC2: LM358MX, linear:LM358MX
- added POT1: RK09K1130A5R, RK09K1130A5R:RK09K1130A5R
- added U$6: 2.1MMJACKTHM, ECE388:2.1MMJACKTHM
- DECREASE, INCREASE: value MOMENTARYBUTTON -> EVP-BFAC1A000; device ECE388:MOMENTARYBUTTON -> EVP-BFAC1A000:EVP-BFAC1A000
- T1: device zetex:PMOSSOT23-6 -> zetex:PMOSSOT23
- U$1: value MCP4921-E/P -> MCP4921-E/SN; device MCP4921-E_P:MCP4921-E/P -> MCP4921-E_SN:MCP4921-E/SN
Connections:
- net +12V: now also IC2P.V+, U$6.TIP; no longer IC3P.V+, J2.PWR
- net +5V: now also POT1.VCC, U$1.!SHDN; no longer R15.A, U$1.VREFA
- net CURRENT_SENSE: now also IC2B.OUT; no longer IC3B.OUT
- net GND: now also DECREASE.A, IC2P.V-, INCREASE.A, POT1.GND, U$6.RING, U$6.RING_SW; no longer DECREASE.A1, IC3P.V-, INCREASE.A1, J2.GND, J2.GNDBREAK, R15.E
- net N$10: now also IC2A.+IN; no longer IC3A.+IN
- net N$12: now also POT1.OUT; no longer R15.S
- net N$16: now also IC2A.OUT; no longer IC3A.OUT
- net N$19: now also IC2A.-IN, IC2B.+IN; no longer IC3A.-IN, IC3B.+IN
- net N$22: now also IC2B.-IN; no longer IC3B.-IN
- net N$23: now also U$1.VOUT; no longer U$1.VOUTA
- net N$6: now also DECREASE.B; no longer DECREASE.B1
- net N$8: now also INCREASE.B; no longer INCREASE.B1
